File: Logic Board(s)/ProtoBlue.brd (EAGLE design)
At the start: 135.9 x 66 mm, 114 parts

Commit message: v2.0.0
Parts:
- removed E$10, E$11, E$12, E$13, E$14, E$15, E$16, E$17, E$20, E$21, E$26, E$28, E$29, E$30, E$31, E$32, E$35, E$37, E$38, E$39, E$40, E$41, E$77, E$78, E$85, E$86, E$87, E$88, E$89, E$90, E$91, E$92, E$93, E$94: (no value), led:LP2C63-ST-RGB-SR0
- removed E$100, E$101, E$110, E$19, E$22, E$46, E$49, E$50, E$51, E$53, E$72, E$95: (no value), eagle-ltspice:0204/7
- removed E$102, E$55, E$56: (no value), v-reg:78MXXS
- removed E$103, E$105, E$107, E$112, E$113, E$114, E$57, E$58, E$61, E$63, E$64, E$66, E$68, E$69, E$70, E$74, E$75, E$76: (no value), eagle-ltspice:LED_SML0603
- removed E$104, E$106, E$27, E$47, E$59, E$60, E$62, E$65, E$99: (no value), eagle-ltspice:R0603
- removed E$108, E$48, E$67: (no value), ref-packages:MINIMELF
- removed E$109, E$52, E$71: (no value), linear:SOT23
- removed E$111, E$54, E$73: (no value), resistor-dil:0603-ARC
- removed E$18, E$7, E$82: (no value), con-lstb:MA03-2
- removed E$23, E$24, E$3, E$36, E$96, E$97: (no value), eagle-ltspice:C0603
- removed E$25, E$45, E$98: (no value), c-trimm:3018_12
- removed E$33, E$4, E$79: (no value), atmel:VQFP32
- removed E$34, E$42, E$5, E$6, E$80, E$81: (no value), switch:TL1105SP
- removed E$43, E$8, E$83: (no value), con-lstb:MA04-2
- removed E$44, E$84, E$9: (no value), crystal:CSM-7X-DU
- added AVR_RES_LED, LED_SW_LED, NRF_EN_SW_LED, NRF_EN_SW_LED1, NRF_TX_SW_LED, RX_LED, SCK_LED, TX_LED: (no value), eagle-ltspice:LED_SML0603
- added AVR_RES_SW: (no value), SparkFun-Switches:TACTILE_SWITCH_SMD_5.2MM
- added AVR_U1: 328AU, atmel:VQFP32
- added AVR_X1, NRF_X1: 16MHz, crystal:CSM-7X-DU
- added AVR_X1_C1, AVR_X1_C2, NRF_X1_C1, NRF_X1_C2: 22pF, ref-packages-longpad:C0603K
- added BTL_U1: ATMEGA8U2-MU, cypress:QFN32
- added BTL_U2: (no value), burr-brown:SO08
- added BTL_U3: LP2985-33DBVR, texas:SOT23-DBV
- added CHG_LED, LED1, LED10, LED11, LED12, LED13, LED14, LED15, LED16, LED17, LED18, LED19, LED2, LED20, LED21, LED22, LED23, LED24, LED3, LED4, LED5, LED6, LED7, LED8, LED9: WS2812B5050, microbuilder:WS2812B-NARROW
- added F1: 500mA, rcl:L1812
- added IC1: MC33269ST-5.0T3, linear:SOT223
- added L1: BLM21, wuerth-elektronik:0805
- added LED_C1, LED_C10, LED_C11, LED_C12, LED_C13, LED_C14, LED_C15, LED_C2, LED_C3, LED_C4, LED_C5, LED_C6, LED_C7, LED_C8, LED_C9: 100nF, rcl:C0603
- added LED_R1: (no value), microbuilder:0603-NO
- added LED_SW, NRF_EN_SW, NRF_TX_SW: (no value), switch:TL1105T
- added NRF_ANT: (no value), con-garry:332-02
- added NRF_C3: 2.2nF, eagle-ltspice:C0603
- added NRF_C4: 4.7pF, eagle-ltspice:C0603
- added NRF_C5: 1.5pF, eagle-ltspice:C0603
- added NRF_C6: 1pF, eagle-ltspice:C0603
- added NRF_C7: 33nF, ref-packages-longpad:C0603K
- added NRF_C8: 1nF, ref-packages-longpad:C0603K
- added NRF_C9: 10nF, ref-packages-longpad:C0603K
- added NRF_L1: 8.2nH, eagle-ltspice:L2012C
- added NRF_L2: 3.9nH, eagle-ltspice:L2012C
- added NRF_L3: 2.7nH, eagle-ltspice:L2012C
- added NRF_R1: 1M, ref-packages-longpad:C0603K
- added NRF_R2: 22K, ref-packages-longpad:C0603K
- added NRF_U1: nRF24L01, allegro:QFN20
- added RN2: 1K, resistor-dil:CAY16
- added RX_R1, TX_R1: 1K, ref-packages-longpad:C0603K
- added SW_RA: 1K, resistor-dil:0603-ARC
- added USB_C1: 47uF, c-trimm:3018_11
- added USB_C2: 100nF, ref-packages-longpad:C0603K
- added USB_D+_R1, USB_D-_R1: 22R, ref-packages-longpad:C0603K
- added USB_Z1, USB_Z2: PGB1010604, ref-packages-longpad:C0603K
- E$1: value (none) -> USB; device led:LP2C63-ST-RGB-SR0 -> con-cypressindustries:32005-400
- E$2: value (none) -> BATT_IN; device led:LP2C63-ST-RGB-SR0 -> SparkFun-Connectors:1X05_1MM_RA
- moved E$1 99.7 mm to (6.00, 35.5), flipped to the bottom
- moved E$2 55.4 mm to (55.0, 31.0), flipped to the bottom, turned to 180 degrees
Connections:
- removed net S$171: E$100.2
- removed net S$174: E$102.IN
- removed net S$175: E$95.2
- removed net S$204: E$95.1
- removed net S$216: E$102.OUT
- removed net S$217: E$100.1
- removed net S$218: E$101.1
- removed net S$219: E$101.2
- removed net S$238: E$102.GND
- new net GND: E$1.5
- new net N$26: LED_R1.1
- new net RXD: AVR_U1.30
- new net RXD1: BTL_U1.8
- new net S$10: SCK_LED.A
- new net S$105: NRF_U1.14
- new net S$12: LED_R1.2
- new net S$13: NRF_U1.6
- new net S$14: AVR_U1.4, AVR_U1.6
- new net S$34: LED2.3-GND
- new net S$86: RX_LED.A
- new net S$91: BTL_U1.10
- new net S$98: BTL_U1.11, TX_LED.C
- new net TXD1: BTL_U1.9
- new net USB_D+: E$1.3
- new net USB_D-: E$1.2
- new net USB_ID: E$1.4
- new net VCC: E$1.1
Routing:
- net S$209: track 228.8 -> 0.00 mm
- net S$177: track 140.5 -> 0.00 mm
- net S$178: track 128.9 -> 0.00 mm
- net S$226: track 91.3 -> 0.00 mm
- net S$216: track 86.4 -> 0.00 mm
- net S$212: track 62.0 -> 0.00 mm
- net S$224: track 59.1 -> 0.00 mm
- net S$228: track 58.3 -> 0.00 mm
- net S$227: track 55.9 -> 0.00 mm
- net S$232: track 46.2 -> 0.00 mm
- net S$231: track 44.1 -> 0.00 mm
- net S$230: track 42.8 -> 0.00 mm
- net S$229: track 41.3 -> 0.00 mm
- net S$179: track 37.5 -> 0.00 mm
- net S$176: track 37.2 -> 0.00 mm
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- removed copper zone on layer 1, net S$253
- removed copper zone on layer 1, net S$254
Other:
- board outline removed
- board text added: "G"
- board text added: "IN"
- board text added: "OUT"
- board text added: "PWR"
- board text added: "RX"
- board text added: "SCK"
- board text added: "TX"
- board text added: "USB"
- board text removed: "MODE"
- board text removed: "VCC"
